File: 13W3.kicad_pcb (KiCad board)
At the start: 2 copper layers, 52 x 53.6 mm, 22 parts, among them J1 DB13W3, J2 VGA, J3 H, J4 V, J5 PWR, U1 LMH1980

Commit message: updated 13w3 connector
updated 13w3 connector to different style
Routing:
- net Net-(J1-PadA1): track 72.3 -> 70.7 mm
- net Net-(J2-Pad3): track 44.1 -> 42.8 mm
- net Net-(J1-PadA2): track 34.9 -> 33.6 mm
